Commit message: Update tri_bot.xacro
Add links and joints for cameras.

File: src/tri_bot_description/urdf/tri_bot.xacro (robot description, xacro)
@@ -7,4 +7,9 @@
   <xacro:property name="tail_length" value="0.2" />
   <xacro:property name="nose_length" value="0.08" />
+  <xacro:property name="zoom_cam_size" value="0.019" />
+  <xacro:property name="night_cam_size_x" value="0.02" />
+  <xacro:property name="night_cam_size_y" value="0.02" />
+  <xacro:property name="night_cam_size_z" value="0.02854" />
+  <xacro:property name="cam_separation" value="0.04" />
   <material name="blue">
     <color rgba="0 0 0.8 1"/>
@@ -15,4 +20,7 @@
   <material name="red">
     <color rgba="0.8 0 0 1"/>
+  </material>
+  <material name="black">
+    <color rgba="0.1 0.1 0.1 1"/>
   </material>
   <link name="base_link">
@@ -29,4 +37,65 @@
     </collision>
   </link>
+  <link name="nose_link">
+    <visual>
+      <geometry>
+        <cone radius="${body_width/2}" length="${nose_length}"/>
+      </geometry>
+      <origin xyz="${nose_length/2} 0 0" rpy="0 1.57 0"/>
+      <material name="blue"/>
+    </visual>
+    <collision>
+      <geometry>
+        <cone radius="${body_width/2}" length="${nose_length}"/>
+      </geometry>
+      <origin xyz="${nose_length/2} 0 0" rpy="0 1.57 0"/>
+    </collision>
+  </link>
+  <joint name="nose_joint" type="fixed">
+    <parent link="base_link"/>
+    <child link="nose_link"/>
+    <origin xyz="${body_length/2} 0 0"/>
+  </joint>
+<link name="camera_night_link">
+    <visual>
+      <geometry>
+        <box size="${night_cam_size_x} ${night_cam_size_y} ${night_cam_size_z}"/>
+      </geometry>
+      <material name="black"/>
+    </visual>
+  </link>
+  <joint name="camera_night_joint" type="fixed">
+    <parent link="nose_link"/>
+    <child link="camera_night_link"/>
+    <origin xyz="${nose_length*0.8} ${cam_separation/2} 0" rpy="0 0 0"/>
+  </joint>
+  <link name="camera_zoom_link">
+    <visual>
+      <geometry>
+        <cylinder radius="${zoom_cam_size/2}" length="${zoom_cam_size*1.5}"/>
+      </geometry>
+      <origin xyz="0 0 0" rpy="0 1.57 0"/>
+      <material name="black"/>
+    </visual>
+  </link>
+  <joint name="camera_zoom_joint" type="fixed">
+    <parent link="nose_link"/>
+    <child link="camera_zoom_link"/>
+    <origin xyz="${nose_length*0.8} -${cam_separation/2} 0" rpy="0 0 0"/>
+  </joint>
+  <!-- ROS 2 and cameras use 2 different coordinate systems -->
+  <!-- The 2 optical frames uniform the standard to the one that ROS 2 uses -->
+  <link name="camera_night_optical_frame"/>
+  <joint name="camera_night_optical_joint" type="fixed">
+    <parent link="camera_night_link"/>
+    <child link="camera_night_optical_frame"/>
+    <origin xyz="0 0 0" rpy="-1.57 0 -1.57"/>
+  </joint>
+  <link name="camera_zoom_optical_frame"/>
+  <joint name="camera_zoom_optical_joint" type="fixed">
+    <parent link="camera_zoom_link"/>
+    <child link="camera_zoom_optical_frame"/>
+    <origin xyz="0 0 0" rpy="-1.57 0 -1.57"/>
+  </joint>
   <link name="left_wing">
     <visual>

Commit message: Update .xacro, CMakeLists.txt, and created display.launch.py Added inertia in .xacro

File: src/tri_bot_description/urdf/tri_bot.xacro (robot description, xacro)
@@ -1,4 +1,33 @@
 <?xml version="1.0"?>
 <robot xmlns:xacro="http://www.ros.org/wiki/xacro" name="tri_bot">
+  <!-- Inertia formulas -->
+  <xacro:macro name="box_inertia" params="m w h d xyz rpy">
+    <inertial>
+      <origin xyz="${xyz}" rpy="${rpy}"/>
+      <mass value="${m}"/>
+      <inertia ixx="${(m/12) * (h*h + d*d)}" ixy="0.0" ixz="0.0"
+               iyy="${(m/12) * (w*w + d*d)}" iyz="0.0"
+               izz="${(m/12) * (w*w + h*h)}"/>
+    </inertial>
+  </xacro:macro>
+  <xacro:macro name="cylinder_inertia" params="m r h xyz rpy">
+    <inertial>
+      <origin xyz="${xyz}" rpy="${rpy}"/>
+      <mass value="${m}"/>
+      <inertia ixx="${(m/12) * (3*r*r + h*h)}" ixy = "0.0" ixz = "0.0"
+               iyy="${(m/12) * (3*r*r + h*h)}" iyz = "0.0"
+               izz="${(m/2) * (r*r)}"/>
+    </inertial>
+  </xacro:macro>
+  <xacro:macro name="sphere_inertia" params="m r xyz rpy">
+    <inertial>
+      <origin xyz="${xyz}" rpy="${rpy}"/>
+      <mass value="${m}"/>
+      <inertia ixx="${(2/5) * m * (r*r)}" ixy="0.0" ixz="0.0"
+               iyy="${(2/5) * m * (r*r)}" iyz="0.0"
+               izz="${(2/5) * m * (r*r)}"/>
+    </inertial>
+  </xacro:macro>
+  <!-- All the values below are approxiamated -->
   <!-- The value indicates the length in meter -->
   <xacro:property name="body_length" value="0.16" />
@@ -36,9 +65,10 @@
       </geometry>
     </collision>
+    <xacro:box_inertia m="3" w="${body_length}" h="${body_width}" d="${body_width}" xyz="0 0 0" rpy="0 0 0"/>
   </link>
   <link name="nose_link">
     <visual>
       <geometry>
-        <cone radius="${body_width/2}" length="${nose_length}"/>
+        <cylinder radius="${body_width/2}" length="${nose_length}"/>
       </geometry>
       <origin xyz="${nose_length/2} 0 0" rpy="0 1.57 0"/>
@@ -47,8 +77,9 @@
     <collision>
       <geometry>
-        <cone radius="${body_width/2}" length="${nose_length}"/>
+        <cylinder radius="${body_width/2}" length="${nose_length}"/>
       </geometry>
       <origin xyz="${nose_length/2} 0 0" rpy="0 1.57 0"/>
     </collision>
+    <xacro:cylinder_inertia m="0.1" r="${body_width/2}" h="${nose_length}" xyz="${nose_length/2} 0 0" rpy="0 1.57 0"/>
   </link>
   <joint name="nose_joint" type="fixed">
@@ -64,4 +95,5 @@
       <material name="black"/>
     </visual>
+    <xacro:box_inertia m="0.01" w="${night_cam_size_x}" h="${night_cam_size_y}" d="${night_cam_size_z}" xyz="0 0 0" rpy="0 0 0"/>
   </link>
   <joint name="camera_night_joint" type="fixed">
@@ -69,4 +101,5 @@
     <child link="camera_night_link"/>
     <origin xyz="${nose_length*0.8} ${cam_separation/2} 0" rpy="0 0 0"/>
+    <xacro:cylinder_inertia m="0.01" r="${zoom_cam_size/2}" h="${zoom_cam_size*1.5}" xyz="0 0 0" rpy="0 1.57 0"/>
   </joint>
   <link name="camera_zoom_link">
@@ -106,4 +139,5 @@
       <material name="blue"/>
     </visual>
+    <xacro:box_inertia m="0.05" w="0.1" h="${single_wing_span}" d="0.02" xyz="0 ${single_wing_span/2} 0" rpy="0 0 0"/>
   </link>
   <joint name="left_wing_fold_joint" type="revolute">
@@ -121,4 +155,5 @@
       <material name="blue"/>
     </visual>
+    <xacro:box_inertia m="0.05" w="0.1" h="${single_wing_span}" d="0.02" xyz="0 -${single_wing_span/2} 0" rpy="0 0 0"/>
   </link>
   <joint name="right_wing_fold_joint" type="revolute">
@@ -136,4 +171,5 @@
       <material name="red"/>
     </visual>
+    <xacro:cylinder_inertia m="0.05" r="0.05" h="${tail_length}" xyz="-${tail_length/2} 0 0" rpy="0 1.57 0"/>
   </link>
   <joint name="tail_mount_joint" type="fixed">
@@ -149,4 +185,5 @@
       <material name="blue"/>
     </visual>
+    <xacro:sphere_inertia m="0.05" r="0.06" xyz="0 0 0" rpy="0 0 0"/>
   </link>
   <joint name="tvc_pitch_joint" type="revolute">

Commit message: Add ros2_control, TVC pitch/yaw, tail fins, ducted fans; align URDF with design
- ros2_control: Add <ros2_control> and gazebo_ros2_control plugin for four
  joints (left/right_wing_fold, tvc_pitch, tvc_yaw). Add config/controllers.yaml
  with JointStateBroadcaster and position_controller (ForwardCommandController). Launch must pass controllers_file:=/path/to/controllers.yaml when using Gazebo.

- TVC: Model spherical joint as pitch + yaw revolute chain (tvc_gimbal_link). Use tvc_range_rad (~30°) for both axes. Document real mechanism: four rods to sliding ball (square vertices), additional rods to rudder; servos drive rods.

- Tail: Replace single rudder with two horizontal tail fins (tail_fin_left/right). Add two counter-rotating ducted fans at tail–body junction (ducted_fan_upper/lower), stacked along z; thrust axis perpendicular to XY (vertical lift). Fully part of tail.

- Nozzle: Visual as bell cylinder + two-bladed propeller; collision and inertia use cylinder (axis x). Add comment on nozzle construction.

- URDF fixes: Remove misplaced inertia from camera_night_joint; add collision to left/right_wing, tail_mount, nozzle; add inertial to camera_zoom_link; cylinder inertia for nozzle instead of sphere.

- controllers.yaml: Rename joint_trajectory_controller to position_controller, add brief comments.

File: src/tri_bot_description/urdf/tri_bot.xacro (robot description, xacro)
@@ -29,5 +29,5 @@
     </inertial>
   </xacro:macro>
-  <!-- All the values below are approxiamated -->
+  <!-- All the values below are approximated -->
   <!-- The value indicates the length in meter -->
   <xacro:property name="body_length" value="0.16" />
@@ -41,4 +41,14 @@
   <xacro:property name="night_cam_size_z" value="0.02854" />
   <xacro:property name="cam_separation" value="0.04" />
+  <xacro:property name="ducted_fan_outer_r" value="0.055" />
+  <xacro:property name="ducted_fan_inner_r" value="0.04" />
+  <xacro:property name="ducted_fan_depth" value="0.03" />
+  <xacro:property name="ducted_fan_z_sep" value="0.06" />
+  <xacro:property name="tail_fin_span" value="0.06" />
+  <xacro:property name="tail_fin_chord" value="0.12" />
+  <xacro:property name="tail_fin_thickness" value="0.008" />
+  <xacro:property name="tail_fin_z_offset" value="0.05" />
+  <!-- TVC: real mechanism uses rods + rudder + 4 spherical attachment points; sliding ball gives ~30 deg cone -->
+  <xacro:property name="tvc_range_rad" value="0.5236" />
   <material name="blue">
     <color rgba="0 0 0.8 1"/>
@@ -67,4 +77,5 @@
     <xacro:box_inertia m="3" w="${body_length}" h="${body_width}" d="${body_width}" xyz="0 0 0" rpy="0 0 0"/>
   </link>
+  <!-- Nose: design has pointed faceted cone; cylinder is a simplified stand-in. -->
   <link name="nose_link">
     <visual>
@@ -88,5 +99,5 @@
     <origin xyz="${body_length/2} 0 0"/>
   </joint>
-<link name="camera_night_link">
+  <link name="camera_night_link">
     <visual>
       <geometry>
@@ -101,5 +112,4 @@
     <child link="camera_night_link"/>
     <origin xyz="${nose_length*0.8} ${cam_separation/2} 0" rpy="0 0 0"/>
-    <xacro:cylinder_inertia m="0.01" r="${zoom_cam_size/2}" h="${zoom_cam_size*1.5}" xyz="0 0 0" rpy="0 1.57 0"/>
   </joint>
   <link name="camera_zoom_link">
@@ -111,4 +121,5 @@
       <material name="black"/>
     </visual>
+    <xacro:box_inertia m="0.01" w="${zoom_cam_size*1.5}" h="${zoom_cam_size}" d="${zoom_cam_size}" xyz="0 0 0" rpy="0 0 0"/>
   </link>
   <joint name="camera_zoom_joint" type="fixed">
@@ -139,4 +150,10 @@
       <material name="blue"/>
     </visual>
+    <collision>
+      <geometry>
+        <box size="0.1 ${single_wing_span} 0.02"/>
+      </geometry>
+      <origin xyz="0 ${single_wing_span/2} 0" rpy="0 0 0"/>
+    </collision>
     <xacro:box_inertia m="0.05" w="0.1" h="${single_wing_span}" d="0.02" xyz="0 ${single_wing_span/2} 0" rpy="0 0 0"/>
   </link>
@@ -155,4 +172,10 @@
       <material name="blue"/>
     </visual>
+    <collision>
+      <geometry>
+        <box size="0.1 ${single_wing_span} 0.02"/>
+      </geometry>
+      <origin xyz="0 -${single_wing_span/2} 0" rpy="0 0 0"/>
+    </collision>
     <xacro:box_inertia m="0.05" w="0.1" h="${single_wing_span}" d="0.02" xyz="0 -${single_wing_span/2} 0" rpy="0 0 0"/>
   </link>
@@ -163,4 +186,9 @@
     <axis xyz="1 0 0"/> <limit lower="0" upper="1.57" effort="10" velocity="1"/>
   </joint>
+  <!-- Tail structure: cylinder mount. Real hardware: a sliding ball carries the tail propeller.
+       Four rods connect the ball to the tail structure; their attachment points on the ball
+       are roughly at the four vertices of a square. Additional rods connect the rudder.
+       Servo motors drive the rods; the ball slides to produce nozzle rotation (~30 deg).
+       Below we model the resulting motion as pitch + yaw revolute joints (equivalent kinematics). -->
   <link name="tail_mount">
     <visual>
@@ -171,4 +199,10 @@
       <material name="red"/>
     </visual>
+    <collision>
+      <geometry>
+        <cylinder length="${tail_length}" radius="0.05"/>
+      </geometry>
+      <origin xyz="-${tail_length/2} 0 0" rpy="0 1.57 0"/>
+    </collision>
     <xacro:cylinder_inertia m="0.05" r="0.05" h="${tail_length}" xyz="-${tail_length/2} 0 0" rpy="0 1.57 0"/>
   </link>
@@ -178,18 +212,181 @@
     <origin xyz="-${body_length/2} 0 0"/>
   </joint>
+  <!-- Two counter-rotating ducted propellers at tail–body junction (stacked up/down); fully part of tail. -->
+  <link name="ducted_fan_upper_link">
+    <visual>
+      <geometry>
+        <cylinder radius="${ducted_fan_outer_r}" length="${ducted_fan_depth}"/>
+      </geometry>
+      <!-- Duct axis along +Z (thrust perpendicular to XY plane) -->
+      <origin xyz="0 0 0" rpy="0 0 0"/>
+      <material name="black"/>
+    </visual>
+    <visual>
+      <geometry>
+        <cylinder radius="${ducted_fan_inner_r}" length="${ducted_fan_depth*1.1}"/>
+      </geometry>
+      <origin xyz="0 0 0" rpy="0 0 0"/>
+      <material name="blue"/>
+    </visual>
+    <collision>
+      <geometry>
+        <cylinder radius="${ducted_fan_outer_r}" length="${ducted_fan_depth}"/>
+      </geometry>
+      <origin xyz="0 0 0" rpy="0 0 0"/>
+    </collision>
+    <xacro:cylinder_inertia m="0.08" r="${ducted_fan_outer_r}" h="${ducted_fan_depth}" xyz="0 0 0" rpy="0 0 0"/>
+  </link>
+  <joint name="ducted_fan_upper_joint" type="fixed">
+    <parent link="tail_mount"/>
+    <child link="ducted_fan_upper_link"/>
+    <origin xyz="0 0 ${ducted_fan_z_sep/2}" rpy="0 0 0"/>
+  </joint>
+  <link name="ducted_fan_lower_link">
+    <visual>
+      <geometry>
+        <cylinder radius="${ducted_fan_outer_r}" length="${ducted_fan_depth}"/>
+      </geometry>
+      <!-- Duct axis along +Z (thrust perpendicular to XY plane) -->
+      <origin xyz="0 0 0" rpy="0 0 0"/>
+      <material name="black"/>
+    </visual>
+    <visual>
+      <geometry>
+        <cylinder radius="${ducted_fan_inner_r}" length="${ducted_fan_depth*1.1}"/>
+      </geometry>
+      <origin xyz="0 0 0" rpy="0 0 0"/>
+      <material name="blue"/>
+    </visual>
+    <collision>
+      <geometry>
+        <cylinder radius="${ducted_fan_outer_r}" length="${ducted_fan_depth}"/>
+      </geometry>
+      <origin xyz="0 0 0" rpy="0 0 0"/>
+    </collision>
+    <xacro:cylinder_inertia m="0.08" r="${ducted_fan_outer_r}" h="${ducted_fan_depth}" xyz="0 0 0" rpy="0 0 0"/>
+  </link>
+  <joint name="ducted_fan_lower_joint" type="fixed">
+    <parent link="tail_mount"/>
+    <child link="ducted_fan_lower_link"/>
+    <origin xyz="0 0 -${ducted_fan_z_sep/2}" rpy="0 0 0"/>
+  </joint>
+  <!-- Two horizontal tail fins (design: symmetric left/right stabilizers on tail boom). -->
+  <link name="tail_fin_left_link">
+    <visual>
+      <geometry>
+        <box size="${tail_fin_chord} ${tail_fin_thickness} ${tail_fin_span}"/>
+      </geometry>
+      <origin xyz="0 0 0" rpy="0 0 0"/>
+      <material name="red"/>
+    </visual>
+    <xacro:box_inertia m="0.01" w="${tail_fin_chord}" h="${tail_fin_thickness}" d="${tail_fin_span}" xyz="0 0 0" rpy="0 0 0"/>
+  </link>
+  <joint name="tail_fin_left_joint" type="fixed">
+    <parent link="tail_mount"/>
+    <child link="tail_fin_left_link"/>
+    <origin xyz="-${tail_length/2} 0 ${tail_fin_z_offset}" rpy="0 0 0"/>
+  </joint>
+  <link name="tail_fin_right_link">
+    <visual>
+      <geometry>
+        <box size="${tail_fin_chord} ${tail_fin_thickness} ${tail_fin_span}"/>
+      </geometry>
+      <origin xyz="0 0 0" rpy="0 0 0"/>
+      <material name="red"/>
+    </visual>
+    <xacro:box_inertia m="0.01" w="${tail_fin_chord}" h="${tail_fin_thickness}" d="${tail_fin_span}" xyz="0 0 0" rpy="0 0 0"/>
+  </link>
+  <joint name="tail_fin_right_joint" type="fixed">
+    <parent link="tail_mount"/>
+    <child link="tail_fin_right_link"/>
+    <origin xyz="-${tail_length/2} 0 -${tail_fin_z_offset}" rpy="0 0 0"/>
+  </joint>
+  <!-- TVC equivalent: pitch + yaw stand in for rods/sliding ball; servo commands map to these joints (30 deg). -->
+  <link name="tvc_gimbal_link">
+    <inertial>
+      <origin xyz="0 0 0" rpy="0 0 0"/>
+      <mass value="0.01"/>
+      <inertia ixx="1e-6" ixy="0" ixz="0" iyy="1e-6" iyz="0" izz="1e-6"/>
+    </inertial>
+  </link>
+  <joint name="tvc_pitch_joint" type="revolute">
+    <parent link="tail_mount"/>
+    <child link="tvc_gimbal_link"/>
+    <origin xyz="-${tail_length} 0 0"/>
+    <axis xyz="0 1 0"/> <limit lower="-${tvc_range_rad}" upper="${tvc_range_rad}" effort="10" velocity="5"/>
+  </joint>
+  <!-- Nozzle: design has bell-shaped housing + two-bladed propeller at rear (TVC joint ahead of this). -->
   <link name="nozzle">
     <visual>
       <geometry>
-        <sphere radius="0.06"/>
-      </geometry>
-      <material name="blue"/>
-    </visual>
-    <xacro:sphere_inertia m="0.05" r="0.06" xyz="0 0 0" rpy="0 0 0"/>
-  </link>
-  <joint name="tvc_pitch_joint" type="revolute">
-    <parent link="tail_mount"/>
+        <cylinder radius="0.06" length="0.04"/>
+      </geometry>
+      <origin xyz="0.02 0 0" rpy="0 1.57 0"/>
+      <material name="blue"/>
+    </visual>
+    <visual>
+      <geometry>
+        <box size="0.005 0.12 0.02"/>
+      </geometry>
+      <origin xyz="0.04 0 0" rpy="0 0 0"/>
+      <material name="black"/>
+    </visual>
+    <visual>
+      <geometry>
+        <box size="0.005 0.02 0.12"/>
+      </geometry>
+      <origin xyz="0.04 0 0" rpy="0 0 0"/>
+      <material name="black"/>
+    </visual>
+    <collision>
+      <geometry>
+        <cylinder radius="0.06" length="0.06"/>
+      </geometry>
+      <origin xyz="0.03 0 0" rpy="0 1.57 0"/>
+    </collision>
+    <!-- Inertia: bell is dominant; use cylinder (axis x) for better accuracy than sphere -->
+    <xacro:cylinder_inertia m="0.05" r="0.06" h="0.06" xyz="0.03 0 0" rpy="0 1.57 0"/>
+  </link>
+  <joint name="tvc_yaw_joint" type="revolute">
+    <parent link="tvc_gimbal_link"/>
     <child link="nozzle"/>
-    <origin xyz="-${tail_length} 0 0"/>
-    <axis xyz="0 1 0"/> <limit lower="-0.5" upper="0.5" effort="10" velocity="5"/>
-  </joint>
+    <origin xyz="0 0 0"/>
+    <axis xyz="0 0 1"/> <limit lower="-${tvc_range_rad}" upper="${tvc_range_rad}" effort="10" velocity="5"/>
+  </joint>
+  <!-- ros2_control: expose joint command/state for Gazebo and real hardware -->
+  <ros2_control name="TriBotControl" type="system">
+    <hardware>
+      <plugin>gazebo_ros2_control/GazeboSystem</plugin>
+    </hardware>
+    <joint name="left_wing_fold_joint">
+      <command_interface name="position"/>
+      <state_interface name="position"/>
+      <state_interface name="velocity"/>
+    </joint>
+    <joint name="right_wing_fold_joint">
+      <command_interface name="position"/>
+      <state_interface name="position"/>
+      <state_interface name="velocity"/>
+    </joint>
+    <joint name="tvc_pitch_joint">
+      <command_interface name="position"/>
+      <state_interface name="position"/>
+      <state_interface name="velocity"/>
+    </joint>
+    <joint name="tvc_yaw_joint">
+      <command_interface name="position"/>
+      <state_interface name="position"/>
+      <state_interface name="velocity"/>
+    </joint>
+  </ros2_control>
+  <!-- Gazebo plugin: load ros2_control controller manager and controllers.
+       When launching in Gazebo, the launch file must pass the absolute path to
+       config/controllers.yaml via: controllers_file:=/path/to/controllers.yaml
+       (e.g. from get_package_share_directory), so the plugin can load it. -->
+  <xacro:property name="controllers_file" value=""/>
+  <gazebo>
+    <plugin name="gazebo_ros2_control" filename="libgazebo_ros2_control.so">
+      <parameters>${controllers_file}</parameters>
+    </plugin>
+  </gazebo>
 </robot>

Commit message: move tail fins to left/right

File: src/tri_bot_description/urdf/tri_bot.xacro (robot description, xacro)
@@ -48,5 +48,6 @@
   <xacro:property name="tail_fin_chord" value="0.12" />
   <xacro:property name="tail_fin_thickness" value="0.008" />
-  <xacro:property name="tail_fin_z_offset" value="0.05" />
+  <!-- tail fins on sides (left/right, Y axis); offset from centerline -->
+  <xacro:property name="tail_fin_y_offset" value="0.04" />
   <!-- TVC: real mechanism uses rods + rudder + 4 spherical attachment points; sliding ball gives ~30 deg cone -->
   <xacro:property name="tvc_range_rad" value="0.5236" />
@@ -285,5 +286,5 @@
     <parent link="tail_mount"/>
     <child link="tail_fin_left_link"/>
-    <origin xyz="-${tail_length/2} 0 ${tail_fin_z_offset}" rpy="0 0 0"/>
+    <origin xyz="-${tail_length/2} -${tail_fin_y_offset} 0" rpy="0 0 0"/>
   </joint>
   <link name="tail_fin_right_link">
@@ -300,5 +301,5 @@
     <parent link="tail_mount"/>
     <child link="tail_fin_right_link"/>
-    <origin xyz="-${tail_length/2} 0 -${tail_fin_z_offset}" rpy="0 0 0"/>
+    <origin xyz="-${tail_length/2} ${tail_fin_y_offset} 0" rpy="0 0 0"/>
   </joint>
   <!-- TVC equivalent: pitch + yaw stand in for rods/sliding ball; servo commands map to these joints (30 deg). -->

Commit message: Fixed Fin Orientation

File: src/tri_bot_description/urdf/tri_bot.xacro (robot description, xacro)
@@ -273,13 +273,14 @@
   </joint>
   <!-- Two horizontal tail fins (design: symmetric left/right stabilizers on tail boom). -->
+  <!-- horizontal tail fin (same orientation as wing: flat in XY, thin in Z) -->
   <link name="tail_fin_left_link">
     <visual>
       <geometry>
-        <box size="${tail_fin_chord} ${tail_fin_thickness} ${tail_fin_span}"/>
+        <box size="${tail_fin_chord} ${tail_fin_span} ${tail_fin_thickness}"/>
       </geometry>
       <origin xyz="0 0 0" rpy="0 0 0"/>
       <material name="red"/>
     </visual>
-    <xacro:box_inertia m="0.01" w="${tail_fin_chord}" h="${tail_fin_thickness}" d="${tail_fin_span}" xyz="0 0 0" rpy="0 0 0"/>
+    <xacro:box_inertia m="0.01" w="${tail_fin_chord}" h="${tail_fin_span}" d="${tail_fin_thickness}" xyz="0 0 0" rpy="0 0 0"/>
   </link>
   <joint name="tail_fin_left_joint" type="fixed">
@@ -291,10 +292,10 @@
     <visual>
       <geometry>
-        <box size="${tail_fin_chord} ${tail_fin_thickness} ${tail_fin_span}"/>
+        <box size="${tail_fin_chord} ${tail_fin_span} ${tail_fin_thickness}"/>
       </geometry>
       <origin xyz="0 0 0" rpy="0 0 0"/>
       <material name="red"/>
     </visual>
-    <xacro:box_inertia m="0.01" w="${tail_fin_chord}" h="${tail_fin_thickness}" d="${tail_fin_span}" xyz="0 0 0" rpy="0 0 0"/>
+    <xacro:box_inertia m="0.01" w="${tail_fin_chord}" h="${tail_fin_span}" d="${tail_fin_thickness}" xyz="0 0 0" rpy="0 0 0"/>
   </link>
   <joint name="tail_fin_right_joint" type="fixed">
