Commit message: Fortress + Harmonic support, use_software_gl for OpenGL

File: src/tri_bot_description/urdf/tri_bot.xacro (robot description, xacro)
@@ -64,4 +64,11 @@
     <color rgba="0.1 0.1 0.1 1"/>
   </material>
+  <!-- Dummy root link (no inertia) for KDL: robot_state_publisher warns if root has inertia -->
+  <link name="base_footprint"/>
+  <joint name="base_footprint_joint" type="fixed">
+    <parent link="base_footprint"/>
+    <child link="base_link"/>
+    <origin xyz="0 0 0" rpy="0 0 0"/>
+  </joint>
   <link name="base_link">
     <visual>
@@ -355,39 +362,74 @@
     <axis xyz="0 0 1"/> <limit lower="-${tvc_range_rad}" upper="${tvc_range_rad}" effort="10" velocity="5"/>
   </joint>
-  <!-- ros2_control: expose joint command/state for Gazebo Harmonic (gz_ros2_control) and real hardware -->
-  <ros2_control name="TriBotControl" type="system">
-    <hardware>
-      <plugin>gz_ros2_control/GazeboSimSystem</plugin>
-    </hardware>
-    <joint name="left_wing_fold_joint">
-      <command_interface name="position"/>
-      <state_interface name="position"/>
-      <state_interface name="velocity"/>
-    </joint>
-    <joint name="right_wing_fold_joint">
-      <command_interface name="position"/>
-      <state_interface name="position"/>
-      <state_interface name="velocity"/>
-    </joint>
-    <joint name="tvc_pitch_joint">
-      <command_interface name="position"/>
-      <state_interface name="position"/>
-      <state_interface name="velocity"/>
-    </joint>
-    <joint name="tvc_yaw_joint">
-      <command_interface name="position"/>
-      <state_interface name="position"/>
-      <state_interface name="velocity"/>
-    </joint>
-  </ros2_control>
-  <!-- Gazebo Harmonic (gz_ros2_control): load controller manager and controllers.
-       Launch must pass controllers_file:=/path/to/controllers.yaml (e.g. from get_package_share_directory). -->
+  <!-- ros2_control: Gazebo Harmonic (gz_ros2_control) or Fortress (ign_ros2_control). Launch: gazebo_fortress:=0 for Harmonic, :=1 for Fortress. -->
+  <xacro:property name="gazebo_fortress" value="0"/>
   <xacro:property name="controllers_file" value=""/>
-  <gazebo>
-    <plugin filename="gz_ros2_control-system" name="gz_ros2_control::GazeboSimROS2ControlPlugin">
-      <robot_param>robot_description</robot_param>
-      <robot_param_node>robot_state_publisher</robot_param_node>
-      <parameters>${controllers_file}</parameters>
-    </plugin>
-  </gazebo>
+  <xacro:unless value="${gazebo_fortress}">
+    <ros2_control name="TriBotControl" type="system">
+      <hardware>
+        <plugin>gz_ros2_control/GazeboSimSystem</plugin>
+      </hardware>
+      <joint name="left_wing_fold_joint">
+        <command_interface name="position"/>
+        <state_interface name="position"/>
+        <state_interface name="velocity"/>
+      </joint>
+      <joint name="right_wing_fold_joint">
+        <command_interface name="position"/>
+        <state_interface name="position"/>
+        <state_interface name="velocity"/>
+      </joint>
+      <joint name="tvc_pitch_joint">
+        <command_interface name="position"/>
+        <state_interface name="position"/>
+        <state_interface name="velocity"/>
+      </joint>
+      <joint name="tvc_yaw_joint">
+        <command_interface name="position"/>
+        <state_interface name="position"/>
+        <state_interface name="velocity"/>
+      </joint>
+    </ros2_control>
+    <gazebo>
+      <plugin filename="gz_ros2_control-system" name="gz_ros2_control::GazeboSimROS2ControlPlugin">
+        <robot_param>robot_description</robot_param>
+        <robot_param_node>robot_state_publisher</robot_param_node>
+        <parameters>${controllers_file}</parameters>
+      </plugin>
+    </gazebo>
+  </xacro:unless>
+  <xacro:if value="${gazebo_fortress}">
+    <ros2_control name="TriBotControl" type="system">
+      <hardware>
+        <plugin>ign_ros2_control/IgnitionSystem</plugin>
+      </hardware>
+      <joint name="left_wing_fold_joint">
+        <command_interface name="position"/>
+        <state_interface name="position"/>
+        <state_interface name="velocity"/>
+      </joint>
+      <joint name="right_wing_fold_joint">
+        <command_interface name="position"/>
+        <state_interface name="position"/>
+        <state_interface name="velocity"/>
+      </joint>
+      <joint name="tvc_pitch_joint">
+        <command_interface name="position"/>
+        <state_interface name="position"/>
+        <state_interface name="velocity"/>
+      </joint>
+      <joint name="tvc_yaw_joint">
+        <command_interface name="position"/>
+        <state_interface name="position"/>
+        <state_interface name="velocity"/>
+      </joint>
+    </ros2_control>
+    <gazebo>
+      <plugin filename="ign_ros2_control-system" name="ign_ros2_control::IgnitionROS2ControlPlugin">
+        <robot_param>robot_description</robot_param>
+        <robot_param_node>robot_state_publisher</robot_param_node>
+        <parameters>${controllers_file}</parameters>
+      </plugin>
+    </gazebo>
+  </xacro:if>
 </robot>

Commit message: Now only support Gazebo Harmonic
Now only support Gazebo Harmonic

File: src/tri_bot_description/urdf/tri_bot.xacro (robot description, xacro)
@@ -362,74 +362,37 @@
     <axis xyz="0 0 1"/> <limit lower="-${tvc_range_rad}" upper="${tvc_range_rad}" effort="10" velocity="5"/>
   </joint>
-  <!-- ros2_control: Gazebo Harmonic (gz_ros2_control) or Fortress (ign_ros2_control). Launch: gazebo_fortress:=0 for Harmonic, :=1 for Fortress. -->
-  <xacro:property name="gazebo_fortress" value="0"/>
+  <!-- ros2_control + gz_ros2_control for Gazebo Harmonic -->
   <xacro:property name="controllers_file" value=""/>
-  <xacro:unless value="${gazebo_fortress}">
-    <ros2_control name="TriBotControl" type="system">
-      <hardware>
-        <plugin>gz_ros2_control/GazeboSimSystem</plugin>
-      </hardware>
-      <joint name="left_wing_fold_joint">
-        <command_interface name="position"/>
-        <state_interface name="position"/>
-        <state_interface name="velocity"/>
-      </joint>
-      <joint name="right_wing_fold_joint">
-        <command_interface name="position"/>
-        <state_interface name="position"/>
-        <state_interface name="velocity"/>
-      </joint>
-      <joint name="tvc_pitch_joint">
-        <command_interface name="position"/>
-        <state_interface name="position"/>
-        <state_interface name="velocity"/>
-      </joint>
-      <joint name="tvc_yaw_joint">
-        <command_interface name="position"/>
-        <state_interface name="position"/>
-        <state_interface name="velocity"/>
-      </joint>
-    </ros2_control>
-    <gazebo>
-      <plugin filename="gz_ros2_control-system" name="gz_ros2_control::GazeboSimROS2ControlPlugin">
-        <robot_param>robot_description</robot_param>
-        <robot_param_node>robot_state_publisher</robot_param_node>
-        <parameters>${controllers_file}</parameters>
-      </plugin>
-    </gazebo>
-  </xacro:unless>
-  <xacro:if value="${gazebo_fortress}">
-    <ros2_control name="TriBotControl" type="system">
-      <hardware>
-        <plugin>ign_ros2_control/IgnitionSystem</plugin>
-      </hardware>
-      <joint name="left_wing_fold_joint">
-        <command_interface name="position"/>
-        <state_interface name="position"/>
-        <state_interface name="velocity"/>
-      </joint>
-      <joint name="right_wing_fold_joint">
-        <command_interface name="position"/>
-        <state_interface name="position"/>
-        <state_interface name="velocity"/>
-      </joint>
-      <joint name="tvc_pitch_joint">
-        <command_interface name="position"/>
-        <state_interface name="position"/>
-        <state_interface name="velocity"/>
-      </joint>
-      <joint name="tvc_yaw_joint">
-        <command_interface name="position"/>
-        <state_interface name="position"/>
-        <state_interface name="velocity"/>
-      </joint>
-    </ros2_control>
-    <gazebo>
-      <plugin filename="ign_ros2_control-system" name="ign_ros2_control::IgnitionROS2ControlPlugin">
-        <robot_param>robot_description</robot_param>
-        <robot_param_node>robot_state_publisher</robot_param_node>
-        <parameters>${controllers_file}</parameters>
-      </plugin>
-    </gazebo>
-  </xacro:if>
+  <ros2_control name="TriBotControl" type="system">
+    <hardware>
+      <plugin>gz_ros2_control/GazeboSimSystem</plugin>
+    </hardware>
+    <joint name="left_wing_fold_joint">
+      <command_interface name="position"/>
+      <state_interface name="position"/>
+      <state_interface name="velocity"/>
+    </joint>
+    <joint name="right_wing_fold_joint">
+      <command_interface name="position"/>
+      <state_interface name="position"/>
+      <state_interface name="velocity"/>
+    </joint>
+    <joint name="tvc_pitch_joint">
+      <command_interface name="position"/>
+      <state_interface name="position"/>
+      <state_interface name="velocity"/>
+    </joint>
+    <joint name="tvc_yaw_joint">
+      <command_interface name="position"/>
+      <state_interface name="position"/>
+      <state_interface name="velocity"/>
+    </joint>
+  </ros2_control>
+  <gazebo>
+    <plugin filename="gz_ros2_control-system" name="gz_ros2_control::GazeboSimROS2ControlPlugin">
+      <robot_param>robot_description</robot_param>
+      <robot_param_node>robot_state_publisher</robot_param_node>
+      <parameters>${controllers_file}</parameters>
+    </plugin>
+  </gazebo>
 </robot>

Commit message: fix(gz_ros2_control): pass controllers_file via xacro arg
- tri_bot.xacro: replace controllers_file property with a xacro arg so the launch-provided controllers_file:=... is not overwritten; fixes gz_ros2_control "empty parameters file" initialization failure.

File: src/tri_bot_description/urdf/tri_bot.xacro (robot description, xacro)
@@ -363,5 +363,5 @@
   </joint>
   <!-- ros2_control + gz_ros2_control for Gazebo Harmonic -->
-  <xacro:property name="controllers_file" value=""/>
+  <xacro:arg name="controllers_file" default=""/>
   <ros2_control name="TriBotControl" type="system">
     <hardware>

Commit message: Enhance simulation health check and position controller test scripts
- Updated check_sim_health.sh to implement a polling mechanism for the controller_manager service, allowing for configurable timeout and polling intervals.
- Modified test_position_controller.sh to clarify the test sequence and ensure TVC channels remain fixed at neutral during the test.
- Adjusted tri_bot.xacro to lock TVC pitch and yaw at neutral, aligning with the V1 MVP assumptions.

File: src/tri_bot_description/urdf/tri_bot.xacro (robot description, xacro)
@@ -323,5 +323,6 @@
     <child link="tvc_gimbal_link"/>
     <origin xyz="-${tail_length} 0 0"/>
-    <axis xyz="0 1 0"/> <limit lower="-${tvc_range_rad}" upper="${tvc_range_rad}" effort="10" velocity="5"/>
+    <!-- V1 MVP: lock TVC pitch at neutral (0 rad). -->
+    <axis xyz="0 1 0"/> <limit lower="0.0" upper="0.0" effort="10" velocity="5"/>
   </joint>
   <!-- Nozzle: design has bell-shaped housing + two-bladed propeller at rear (TVC joint ahead of this). -->
@@ -360,5 +361,6 @@
     <child link="nozzle"/>
     <origin xyz="0 0 0"/>
-    <axis xyz="0 0 1"/> <limit lower="-${tvc_range_rad}" upper="${tvc_range_rad}" effort="10" velocity="5"/>
+    <!-- V1 MVP: lock TVC yaw at neutral (0 rad). -->
+    <axis xyz="0 0 1"/> <limit lower="0.0" upper="0.0" effort="10" velocity="5"/>
   </joint>
   <!-- ros2_control + gz_ros2_control for Gazebo Harmonic -->

Commit message: Enhance tri_bot simulation scripts and URDF configuration
- Updated check_sim_health.sh to improve service availability checks for controller_manager.
- Modified start_sim.sh to prevent duplicate simulation launches by checking for existing controller_manager services.
- Enhanced TvcAllocatorNode in tvc_allocator.cpp to allow configurable output topic for position commands.
- Added installation of mesh assets in CMakeLists.txt for URDF visuals.
- Updated gazebo.launch.py to include a new launch argument for rendering debug frames.
- Introduced debug origin markers in tri_bot.xacro for visualizing key link/joint origins in Gazebo.

File: src/tri_bot_description/urdf/tri_bot.xacro (robot description, xacro)
@@ -28,4 +28,22 @@
                izz="${(2/5) * m * (r*r)}"/>
     </inertial>
+  </xacro:macro>
+  <!-- Debug visual marker for checking frame origins in Gazebo. -->
+  <xacro:macro name="debug_origin_marker" params="name parent xyz rpy radius rgba">
+    <link name="${name}">
+      <visual>
+        <geometry>
+          <sphere radius="${radius}"/>
+        </geometry>
+        <material>
+          <color rgba="${rgba}"/>
+        </material>
+      </visual>
+    </link>
+    <joint name="${name}_joint" type="fixed">
+      <parent link="${parent}"/>
+      <child link="${name}"/>
+      <origin xyz="${xyz}" rpy="${rpy}"/>
+    </joint>
   </xacro:macro>
   <!-- All the values below are approximated -->
@@ -178,5 +196,5 @@
       </geometry>
       <origin xyz="0 -${single_wing_span/2} 0" rpy="0 0 0"/>
-      <material name="blue"/>
+      <material name="red"/>
     </visual>
     <collision>
@@ -364,4 +382,53 @@
     <axis xyz="0 0 1"/> <limit lower="0.0" upper="0.0" effort="10" velocity="5"/>
   </joint>
+  <!-- Optional debug markers for key link/joint origins in Gazebo. -->
+  <xacro:arg name="show_debug_frames" default="false"/>
+  <xacro:if value="$(arg show_debug_frames)">
+    <!-- base_link origin -->
+    <xacro:debug_origin_marker
+      name="dbg_base_link_origin"
+      parent="base_link"
+      xyz="0 0 0"
+      rpy="0 0 0"
+      radius="0.012"
+      rgba="1 1 0 1"/>
+    <!-- wing fold joint origins (in base_link frame) -->
+    <xacro:debug_origin_marker
+      name="dbg_left_wing_joint_origin"
+      parent="base_link"
+      xyz="0.05 ${body_width/2} 0"
+      rpy="0 0 0"
+      radius="0.010"
+      rgba="0 0 1 1"/>
+    <xacro:debug_origin_marker
+      name="dbg_right_wing_joint_origin"
+      parent="base_link"
+      xyz="0.05 -${body_width/2} 0"
+      rpy="0 0 0"
+      radius="0.010"
+      rgba="1 0 0 1"/>
+    <!-- tail and TVC joint origins -->
+    <xacro:debug_origin_marker
+      name="dbg_tail_mount_joint_origin"
+      parent="base_link"
+      xyz="-${body_length/2} 0 0"
+      rpy="0 0 0"
+      radius="0.010"
+      rgba="1 0 1 1"/>
+    <xacro:debug_origin_marker
+      name="dbg_tvc_pitch_joint_origin"
+      parent="tail_mount"
+      xyz="-${tail_length} 0 0"
+      rpy="0 0 0"
+      radius="0.009"
+      rgba="0 1 1 1"/>
+    <xacro:debug_origin_marker
+      name="dbg_tvc_yaw_joint_origin"
+      parent="tvc_gimbal_link"
+      xyz="0 0 0"
+      rpy="0 0 0"
+      radius="0.009"
+      rgba="0 1 0 1"/>
+  </xacro:if>
   <!-- ros2_control + gz_ros2_control for Gazebo Harmonic -->
   <xacro:arg name="controllers_file" default=""/>
