Commit message: Integrate Ardupilot and add wings mesh to .xacro
- Updated start_sim.sh to support software rendering and improved error handling for workspace and ArduPilot directory checks.
- Modified CMakeLists.txt to install mesh assets for URDF visuals.
- Refined gazebo.launch.py to utilize the native gz CLI for spawning entities and removed unnecessary debug frame options.
- Updated tri_bot.xacro to include an IMU sensor and adjusted joint configurations for better simulation fidelity.

File: src/tri_bot_description/urdf/tri_bot.xacro (robot description, xacro)
@@ -28,22 +28,4 @@
                izz="${(2/5) * m * (r*r)}"/>
     </inertial>
-  </xacro:macro>
-  <!-- Debug visual marker for checking frame origins in Gazebo. -->
-  <xacro:macro name="debug_origin_marker" params="name parent xyz rpy radius rgba">
-    <link name="${name}">
-      <visual>
-        <geometry>
-          <sphere radius="${radius}"/>
-        </geometry>
-        <material>
-          <color rgba="${rgba}"/>
-        </material>
-      </visual>
-    </link>
-    <joint name="${name}_joint" type="fixed">
-      <parent link="${parent}"/>
-      <child link="${name}"/>
-      <origin xyz="${xyz}" rpy="${rpy}"/>
-    </joint>
   </xacro:macro>
   <!-- All the values below are approximated -->
@@ -91,6 +73,7 @@
   <link name="base_link">
     <visual>
-      <geometry>
-        <box size="${body_length} ${body_width} ${body_width}"/>
+      <origin xyz="0 0 0" rpy="0 0 0"/>
+      <geometry>
+        <mesh filename="package://tri_bot_description/mesh/EUN1_V7_fuselage_1.STL" scale="0.001 0.001 0.001"/>
       </geometry>
       <material name="white"/>
@@ -171,29 +154,30 @@
     <visual>
       <geometry>
+        <mesh filename="package://tri_bot_description/mesh/EUN1_V7_left_wing.STL" scale="0.001 0.001 0.001"/>
+      </geometry>
+      <origin xyz="0 0 0" rpy="0 0 0"/>
+      <material name="blue"/>
+    </visual>
+    <collision>
+      <geometry>
         <box size="0.1 ${single_wing_span} 0.02"/>
       </geometry>
       <origin xyz="0 ${single_wing_span/2} 0" rpy="0 0 0"/>
-      <material name="blue"/>
-    </visual>
-    <collision>
-      <geometry>
-        <box size="0.1 ${single_wing_span} 0.02"/>
-      </geometry>
-      <origin xyz="0 ${single_wing_span/2} 0" rpy="0 0 0"/>
     </collision>
     <xacro:box_inertia m="0.05" w="0.1" h="${single_wing_span}" d="0.02" xyz="0 ${single_wing_span/2} 0" rpy="0 0 0"/>
   </link>
-  <joint name="left_wing_fold_joint" type="revolute">
+  <joint name="left_wing_fold_joint" type="fixed">
     <parent link="base_link"/>
     <child link="left_wing"/>
-    <origin xyz="0.05 ${body_width/2} 0"/>
-    <axis xyz="1 0 0"/> <limit lower="-1.57" upper="0" effort="10" velocity="1"/>
+    <origin xyz="0 0 0"/>
+    <!-- <axis xyz="1 0 0"/> <limit lower="-1.57" upper="0" effort="10" velocity="1"/>
+    <dynamics damping="5.0"/> -->
   </joint>
   <link name="right_wing">
     <visual>
       <geometry>
-        <box size="0.1 ${single_wing_span} 0.02"/>
-      </geometry>
-      <origin xyz="0 -${single_wing_span/2} 0" rpy="0 0 0"/>
+        <mesh filename="package://tri_bot_description/mesh/EUN1_V7_right_wing.STL" scale="0.001 0.001 0.001"/>
+      </geometry>
+      <origin xyz="0.00651 -0.0835 0.02567" rpy="0 0 0"/>
       <material name="red"/>
     </visual>
@@ -209,6 +193,7 @@
     <parent link="base_link"/>
     <child link="right_wing"/>
-    <origin xyz="0.05 -${body_width/2} 0"/>
+    <origin xyz="0 0 0"/>
     <axis xyz="1 0 0"/> <limit lower="0" upper="1.57" effort="10" velocity="1"/>
+    <dynamics damping="5.0"/>
   </joint>
   <!-- Tail structure: cylinder mount. Real hardware: a sliding ball carries the tail propeller.
@@ -341,6 +326,5 @@
     <child link="tvc_gimbal_link"/>
     <origin xyz="-${tail_length} 0 0"/>
-    <!-- V1 MVP: lock TVC pitch at neutral (0 rad). -->
-    <axis xyz="0 1 0"/> <limit lower="0.0" upper="0.0" effort="10" velocity="5"/>
+    <axis xyz="0 1 0"/> <limit lower="-${tvc_range_rad}" upper="${tvc_range_rad}" effort="10" velocity="5"/>
   </joint>
   <!-- Nozzle: design has bell-shaped housing + two-bladed propeller at rear (TVC joint ahead of this). -->
@@ -379,89 +363,196 @@
     <child link="nozzle"/>
     <origin xyz="0 0 0"/>
-    <!-- V1 MVP: lock TVC yaw at neutral (0 rad). -->
-    <axis xyz="0 0 1"/> <limit lower="0.0" upper="0.0" effort="10" velocity="5"/>
-  </joint>
-  <!-- Optional debug markers for key link/joint origins in Gazebo. -->
-  <xacro:arg name="show_debug_frames" default="false"/>
-  <xacro:if value="$(arg show_debug_frames)">
-    <!-- base_link origin -->
-    <xacro:debug_origin_marker
-      name="dbg_base_link_origin"
-      parent="base_link"
-      xyz="0 0 0"
-      rpy="0 0 0"
-      radius="0.012"
-      rgba="1 1 0 1"/>
-    <!-- wing fold joint origins (in base_link frame) -->
-    <xacro:debug_origin_marker
-      name="dbg_left_wing_joint_origin"
-      parent="base_link"
-      xyz="0.05 ${body_width/2} 0"
-      rpy="0 0 0"
-      radius="0.010"
-      rgba="0 0 1 1"/>
-    <xacro:debug_origin_marker
-      name="dbg_right_wing_joint_origin"
-      parent="base_link"
-      xyz="0.05 -${body_width/2} 0"
-      rpy="0 0 0"
-      radius="0.010"
-      rgba="1 0 0 1"/>
-    <!-- tail and TVC joint origins -->
-    <xacro:debug_origin_marker
-      name="dbg_tail_mount_joint_origin"
-      parent="base_link"
-      xyz="-${body_length/2} 0 0"
-      rpy="0 0 0"
-      radius="0.010"
-      rgba="1 0 1 1"/>
-    <xacro:debug_origin_marker
-      name="dbg_tvc_pitch_joint_origin"
-      parent="tail_mount"
-      xyz="-${tail_length} 0 0"
-      rpy="0 0 0"
-      radius="0.009"
-      rgba="0 1 1 1"/>
-    <xacro:debug_origin_marker
-      name="dbg_tvc_yaw_joint_origin"
-      parent="tvc_gimbal_link"
-      xyz="0 0 0"
-      rpy="0 0 0"
-      radius="0.009"
-      rgba="0 1 0 1"/>
+    <axis xyz="0 0 1"/> <limit lower="-${tvc_range_rad}" upper="${tvc_range_rad}" effort="10" velocity="5"/>
+  </joint>
+  <!-- IMU sensor on base_link (required by ArduPilotPlugin and useful for ROS 2). -->
+  <link name="imu_link">
+    <inertial>
+      <mass value="0.01"/>
+      <inertia ixx="1e-7" ixy="0" ixz="0" iyy="1e-7" iyz="0" izz="1e-7"/>
+    </inertial>
+  </link>
+  <joint name="imu_joint" type="revolute">
+    <parent link="base_link"/>
+    <child link="imu_link"/>
+    <origin xyz="0 0 0" rpy="0 0 0"/>
+    <axis xyz="0 0 1"/>
+    <limit lower="0" upper="0" effort="0" velocity="0"/>
+    <dynamics damping="1.0"/>
+  </joint>
+  <gazebo reference="imu_link">
+    <sensor name="imu_sensor" type="imu">
+      <pose degrees="true">0 0 0 180 0 0</pose>
+      <always_on>1</always_on>
+      <update_rate>1000</update_rate>
+    </sensor>
+  </gazebo>
+  <!-- ======= Control back-end selection =======
+       use_ardupilot:=false  (default) → gz_ros2_control path
+       use_ardupilot:=true              → ArduPilotPlugin path (for SITL) -->
+  <xacro:arg name="use_ardupilot" default="false"/>
+  <!-- ── ROS 2 control path ─────────────────────────────────────────── -->
+  <xacro:unless value="$(arg use_ardupilot)">
+    <xacro:arg name="controllers_file" default=""/>
+    <ros2_control name="TriBotControl" type="system">
+      <hardware>
+        <plugin>gz_ros2_control/GazeboSimSystem</plugin>
+      </hardware>
+      <joint name="left_wing_fold_joint">
+        <command_interface name="position"/>
+        <state_interface name="position"/>
+        <state_interface name="velocity"/>
+      </joint>
+      <joint name="right_wing_fold_joint">
+        <command_interface name="position"/>
+        <state_interface name="position"/>
+        <state_interface name="velocity"/>
+      </joint>
+      <joint name="tvc_pitch_joint">
+        <command_interface name="position"/>
+        <state_interface name="position"/>
+        <state_interface name="velocity"/>
+      </joint>
+      <joint name="tvc_yaw_joint">
+        <command_interface name="position"/>
+        <state_interface name="position"/>
+        <state_interface name="velocity"/>
+      </joint>
+    </ros2_control>
+    <gazebo>
+      <plugin filename="gz_ros2_control-system" name="gz_ros2_control::GazeboSimROS2ControlPlugin">
+        <robot_param>robot_description</robot_param>
+        <robot_param_node>robot_state_publisher</robot_param_node>
+        <parameters>$(arg controllers_file)</parameters>
+      </plugin>
+    </gazebo>
+  </xacro:unless>
+  <!-- ── ArduPilot SITL path ─────────────────────────────────────────── -->
+  <xacro:if value="$(arg use_ardupilot)">
+    <gazebo>
+      <plugin name="ArduPilotPlugin" filename="ArduPilotPlugin">
+        <fdm_addr>127.0.0.1</fdm_addr>
+        <fdm_port_in>9002</fdm_port_in>
+        <connectionTimeoutMaxCount>5</connectionTimeoutMaxCount>
+        <lock_step>1</lock_step>
+        <!-- tri_bot body frame: X-forward, Y-left, Z-up (ROS REP-103).
+             ArduPilot NED: X-forward, Y-right, Z-down.
+             Rotation from Gazebo model frame to ArduPilot body: 180 deg roll. -->
+        <modelXYZToAirplaneXForwardZDown degrees="true">0 0 0 180 0 0</modelXYZToAirplaneXForwardZDown>
+        <gazeboXYZToNED degrees="true">0 0 0 180 0 90</gazeboXYZToNED>
+        <imuName>imu_link::imu_sensor</imuName>
+        <!-- CH1 (SERVO1): left wing fold — POSITION servo -->
+        <control channel="0">
+          <jointName>left_wing_fold_joint</jointName>
+          <useForce>1</useForce>
+          <multiplier>-3.14</multiplier>
+          <offset>-0.5</offset>
+          <servo_min>1100</servo_min>
+          <servo_max>1900</servo_max>
+          <type>POSITION</type>
+          <p_gain>10.0</p_gain>
+          <i_gain>0</i_gain>
+          <d_gain>0</d_gain>
+          <i_max>0</i_max>
+          <i_min>0</i_min>
+          <cmd_max>0.0</cmd_max>
+          <cmd_min>-1.57</cmd_min>
+        </control>
+        <!-- CH2 (SERVO2): right wing fold — POSITION servo -->
+        <control channel="1">
+          <jointName>right_wing_fold_joint</jointName>
+          <useForce>1</useForce>
+          <multiplier>3.14</multiplier>
+          <offset>-0.5</offset>
+          <servo_min>1100</servo_min>
+          <servo_max>1900</servo_max>
+          <type>POSITION</type>
+          <p_gain>10.0</p_gain>
+          <i_gain>0</i_gain>
+          <d_gain>0</d_gain>
+          <i_max>0</i_max>
+          <i_min>0</i_min>
+          <cmd_max>1.57</cmd_max>
+          <cmd_min>0.0</cmd_min>
+        </control>
+        <!-- CH3 (SERVO3): throttle — maps to nozzle joint velocity as a stand-in for thrust -->
+        <control channel="2">
+          <jointName>tvc_yaw_joint</jointName>
+          <useForce>0</useForce>
+          <multiplier>0</multiplier>
+          <offset>0</offset>
+          <servo_min>1100</servo_min>
+          <servo_max>1900</servo_max>
+          <type>VELOCITY</type>
+          <p_gain>0</p_gain>
+          <i_gain>0</i_gain>
+          <d_gain>0</d_gain>
+          <i_max>0</i_max>
+          <i_min>0</i_min>
+          <cmd_max>0</cmd_max>
+          <cmd_min>0</cmd_min>
+        </control>
+        <!-- CH4 (SERVO4): TVC pitch — POSITION servo -->
+        <control channel="3">
+          <jointName>tvc_pitch_joint</jointName>
+          <useForce>1</useForce>
+          <multiplier>-1.048</multiplier>
+          <offset>-0.5</offset>
+          <servo_min>1100</servo_min>
+          <servo_max>1900</servo_max>
+          <type>POSITION</type>
+          <p_gain>10.0</p_gain>
+          <i_gain>0</i_gain>
+          <d_gain>0</d_gain>
+          <i_max>0</i_max>
+          <i_min>0</i_min>
+          <cmd_max>0.524</cmd_max>
+          <cmd_min>-0.524</cmd_min>
+        </control>
+        <!-- CH5 (SERVO5): TVC yaw — POSITION servo -->
+        <control channel="4">
+          <jointName>tvc_yaw_joint</jointName>
+          <useForce>1</useForce>
+          <multiplier>-1.048</multiplier>
+          <offset>-0.5</offset>
+          <servo_min>1100</servo_min>
+          <servo_max>1900</servo_max>
+          <type>POSITION</type>
+          <p_gain>10.0</p_gain>
+          <i_gain>0</i_gain>
+          <d_gain>0</d_gain>
+          <i_max>0</i_max>
+          <i_min>0</i_min>
+          <cmd_max>0.524</cmd_max>
+          <cmd_min>-0.524</cmd_min>
+        </control>
+      </plugin>
+    </gazebo>
+    <!-- Publish joint states so ArduPilotPlugin can read JointPosition components -->
+    <gazebo>
+      <plugin filename="gz-sim-joint-state-publisher-system"
+        name="gz::sim::systems::JointStatePublisher">
+      </plugin>
+    </gazebo>
+    <!-- ApplyJointForce required for each joint ArduPilot drives -->
+    <gazebo>
+      <plugin filename="gz-sim-apply-joint-force-system" name="gz::sim::systems::ApplyJointForce">
+        <joint_name>left_wing_fold_joint</joint_name>
+      </plugin>
+    </gazebo>
+    <gazebo>
+      <plugin filename="gz-sim-apply-joint-force-system" name="gz::sim::systems::ApplyJointForce">
+        <joint_name>right_wing_fold_joint</joint_name>
+      </plugin>
+    </gazebo>
+    <gazebo>
+      <plugin filename="gz-sim-apply-joint-force-system" name="gz::sim::systems::ApplyJointForce">
+        <joint_name>tvc_pitch_joint</joint_name>
+      </plugin>
+    </gazebo>
+    <gazebo>
+      <plugin filename="gz-sim-apply-joint-force-system" name="gz::sim::systems::ApplyJointForce">
+        <joint_name>tvc_yaw_joint</joint_name>
+      </plugin>
+    </gazebo>
   </xacro:if>
-  <!-- ros2_control + gz_ros2_control for Gazebo Harmonic -->
-  <xacro:arg name="controllers_file" default=""/>
-  <ros2_control name="TriBotControl" type="system">
-    <hardware>
-      <plugin>gz_ros2_control/GazeboSimSystem</plugin>
-    </hardware>
-    <joint name="left_wing_fold_joint">
-      <command_interface name="position"/>
-      <state_interface name="position"/>
-      <state_interface name="velocity"/>
-    </joint>
-    <joint name="right_wing_fold_joint">
-      <command_interface name="position"/>
-      <state_interface name="position"/>
-      <state_interface name="velocity"/>
-    </joint>
-    <joint name="tvc_pitch_joint">
-      <command_interface name="position"/>
-      <state_interface name="position"/>
-      <state_interface name="velocity"/>
-    </joint>
-    <joint name="tvc_yaw_joint">
-      <command_interface name="position"/>
-      <state_interface name="position"/>
-      <state_interface name="velocity"/>
-    </joint>
-  </ros2_control>
-  <gazebo>
-    <plugin filename="gz_ros2_control-system" name="gz_ros2_control::GazeboSimROS2ControlPlugin">
-      <robot_param>robot_description</robot_param>
-      <robot_param_node>robot_state_publisher</robot_param_node>
-      <parameters>$(arg controllers_file)</parameters>
-    </plugin>
-  </gazebo>
 </robot>
